File: carrier.kicad_sch (KiCad schematic)
At the start: 44 parts, among them U2 STM32C071G8Ux, U3 TPS7A20xxxDBV, U4 TPS7A20xxxDBV, U5 TPS7A20xxxDBV

Commit message: schematic complete
Parts:
- removed C20, C21, C22, C23, C24, C25: 10uF, ar_passives:C_0805, symbol #bt-db:capacitor/CAPC-00926
- removed C5: 470nF, ar_passives:C_0402, symbol #bt-db:capacitor/CAPC-00613
- removed C6: 100nF, ar_passives:C_0402, symbol #bt-db:capacitor/CAPC-00573
- removed C9: 10nF, ar_passives:C_0402, symbol #bt-db:capacitor/CAPC-00514
- removed U3, U4, U5: TPS7A20xxxDBV, Package_TO_SOT_SMD:SOT-23-5, symbol Regulator_Linear:TPS7A20xxxDBV
- added C20, C34, C37, C40: 1uF, ar_passives:C_0402, symbol #bt-db:capacitor/CAPC-00622
- added C21, C22, C23, C24, C36: 100nF, ar_passives:C_0402, symbol #bt-db:capacitor/CAPC-00573
- added C25, C9: 10uF, ar_passives:C_0402, symbol #bt-db:capacitor/CAPC-00667
- added C26, C27, C28, C29, C30, C31, C32, C33, C35: 10uF, ar_passives:C_0805, symbol #bt-db:capacitor/CAPC-00926
- added D1, D2, D3: Green, ar_opto:LED_0603, symbol #bt-db:optical/LEDO-00006
- added D4: Red, ar_opto:LED_0603, symbol #bt-db:optical/LEDO-00004
- added D5: (no value), ar_discrete:SOD123W, symbol #bt-db:diode/DIOD-00060
- added F1: 0.5A, ar_passives:F_1210, symbol #bt-db:fuse/FUSE-00006
- added J1, J2, J3, J4, J7, J8: 732511151, ar_connector:Molex 73251-1151, symbol #bt-db:connector/CONN-00215
- added J5: FTSH-105-01-L-DV-K, ar_connector:FTSH-105-01-X-DV-K, symbol #bt-db:connector/CONN-00005
- added J6: USB4110-GF-A, ar_connector:USB-C USB4110, symbol #bt-db:connector/CONN-00188
- added J9: M20-9990445, ar_connector:Header 2.54 1x04 Staggered, symbol #bt-db:connector/CONN-00026
- added L1: 1uH, ar_passives:L_252010, symbol #bt-db:inductor/INDU-00044
- added R10: 44.2k, ar_passives:R_0402, symbol #bt-db:resistor/RESI-01263
- added R11, R12, R13, R14: 1k, ar_passives:R_0402, symbol #bt-db:resistor/RESI-01054
- added R15, R16, R21, R22: 5.11k, ar_passives:R_0402, symbol #bt-db:resistor/RESI-01142
- added R17, R18, R19, R20: 0R, ar_passives:R_0402, symbol #bt-db:resistor/RESI-00694
- added R9: 200k, ar_passives:R_0402, symbol #bt-db:resistor/RESI-01352
- added TP1: SCK, ar_non-bom:Testpad_1mm, symbol Connector:TestPoint
- added TP10, TP11, TP9: SDA, ar_non-bom:Testpad_1mm, symbol Connector:TestPoint
- added TP2: MUX, ar_non-bom:Testpad_1mm, symbol Connector:TestPoint
- added TP3: SDI, ar_non-bom:Testpad_1mm, symbol Connector:TestPoint
- added TP4: RC, ar_non-bom:Testpad_1mm, symbol Connector:TestPoint
- added TP5: RD, ar_non-bom:Testpad_1mm, symbol Connector:TestPoint
- added TP6: CE, ar_non-bom:Testpad_1mm, symbol Connector:TestPoint
- added TP7: CS, ar_non-bom:Testpad_1mm, symbol Connector:TestPoint
- added TP8: SCL, ar_non-bom:Testpad_1mm, symbol Connector:TestPoint
- added U3: (no value), ar_ic:SOT-23-3, symbol #bt-db:ic/ICIR-00100
- added U4: (no value), ar_ic:DFN6-1.55x1.75, symbol #bt-db:ic/ICIR-00298
- added U6: (no value), ar_ic:SOT563, symbol #bt-db:ic/ICIR-00044
- added Y2: 38.4MHz, ar_passives:XTAL2016-4, symbol #bt-db:crystal/XTAL-00014
Connections:
- net 3V3_BUF: now also C23.1, C24.1, C33.1; no longer R3.1
- net 3V3_SYN: no longer R1.1
- net GND: now also U2.4 (VSS), C20.2, C21.2, C22.2, C23.2, C24.2, C25.2, C26.2, C27.2, C28.2, C29.2, C30.2, C31.2, C32.2, C33.2, C34.2, C35.2, C36.2, C37.2, C40.2, C9.2, D1.K, D2.K, D3.K, D4.K, D5.A, J1.outer (Outer), J2.outer (Outer), J3.outer (Outer), J4.outer (Outer), J5.3, J5.5, J5.7, J5.9, J6.A1-B12 (GND), J6.A12-B1 (GND), J6.SH (Shield), J7.outer (Outer), J8.outer (Outer), J9.1, R10.2, R15.2, R16.2, U3.1 (GND), U4.3 (GND), U6.2 (GND), Y2.2 (GND)
- net SYN.CE: now also U2.28 (PB8), TP6.1
- net SYN.MUX: now also U2.24 (PB4), TP2.1
- net SYN.RC: now also U2.26 (PB6), TP4.1
- net SYN.RD: now also U2.27 (PB7), TP5.1
- net SYN.SCK: now also U2.23 (PB3), TP1.1
- net SYN.SDI: now also U2.25 (PB5), TP3.1
- net SYN.~{CS}: now also U2.22 (PA15), TP7.1
- net VbiasVCO: now also C9.1
- net VbiasVCO2: now also C25.1
- net VregVCO: now also C34.1
- net MCU_REF_IN: now reaches U2.1 (PC14)
- net LED_ERR: now reaches U2.10 (PA4)
- net LED_ERR: now also R14.1
- net OLED_SDA: now reaches U2.12 (PA6)
- net OLED_SDA: now also J9.4, R21.2, TP9.1
- net OLED_SCL: now reaches U2.13 (PA7)
- net OLED_SCL: now also J9.3, R22.2, TP8.1
- net BUCK_EN: now reaches U2.14 (PB0)
- net BUCK_EN: now also U6.5 (EN)
- net USB_DN: now reaches U2.18 (PA11)
- net USB_DN: now also U4.1 (CON+)
- net USB_DP: now reaches U2.19 (PA12)
- net USB_DP: now also U4.2 (CON-)
- net DBG_SWDIO: now reaches U2.20 (PA13)
- net DBG_SWDIO: now also J5.2
- net DBG_SWCLK: now reaches U2.21 (PA14)
- net DBG_SWCLK: now also J5.4
- net 3V3_MCU: now reaches U2.3 (VDD)
- net 3V3_MCU: now also C20.1, C21.1, C22.1, C32.1, C37.1, J5.1, J9.2, R11.1, R21.1, R22.1, U3.2 (OUT)
- net ~{DBG_NRST}: now reaches U2.5 (PF2)
- net ~{DBG_NRST}: now also J5.10
- net DBG_TX: now reaches U2.6 (PA0)
- net DBG_TX: now also J5.6, TP11.1
- net DBG_RX: now reaches U2.7 (PA1)
- net DBG_RX: now also J5.8, TP10.1
- net LED_STAT: now reaches U2.9 (PA3)
- net LED_STAT: now also R13.1
- net LO_A.N renamed SMA_A_N
- net SMA_A_N: now also J2.inner (Inner)
- net LO_A.P renamed SMA_A_P
- net SMA_A_P: now also J1.inner (Inner)
- net LO_B.N renamed SMA_B_N
- net SMA_B_N: now also J4.inner (Inner)
- net LO_B.P renamed SMA_B_P
- net SMA_B_P: now also J3.inner (Inner)
- net REF.N renamed REF_N
- net REF_N: now also R19.2
- net REF.P renamed REF_P
- net REF_P: now also R18.2, R20.2
- new net: J6.B5 (CC2), R16.1
- new net: F1.1, J6.A4-B9 (VBUS), J6.A9-B4 (VBUS)
- new net: D3.A, R13.2
- new net: D1.A, R11.2
- new net: R10.1, R9.2, U6.1 (FB)
- new net: L1.1, U6.4 (SW)
- new net: J6.A5 (CC1), R15.1
- new net: D4.A, R14.2
- new net: D2.A, R12.2
- new net 3V3_BUCK: C26.1, C28.1, C29.1, C30.1, L1.2, R1.1, R12.1, R17.1, R3.1, R9.1, U6.6 (OUT)
- new net 3V3_OSC: C35.1, C36.1, C40.1, R17.2, Y2.4 (VCC)
- new net CON_DN: J6.A7 (D-), J6.B7 (D-), U4.6 (IC+)
- new net CON_DP: J6.A6 (D+), J6.B6 (D+), U4.5 (IC-)
- new net REF_SMA_N: J7.inner (Inner), R19.1
- new net REF_SMA_P: J8.inner (Inner), R20.1
- new net REF_TCXO: R18.1, Y2.3 (OUT)
- new net VBUS: C27.1, C31.1, D5.K, F1.2, U3.3 (IN), U6.3 (VIN)
- no-connect marks 2 -> 6
Other:
- moved on the sheet: C1, C10, C11, C12, C13, C14, C15, C16, C17, C18, C19, C2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
