File: bak/carrier.kicad_sch (KiCad schematic)
At the start: 105 parts, among them J1 USB4110-GF-A, J10 TC2030-NL-FP, J2 732511151, J3 732511151, J4 732511151, J5 732511151, J6 732511151, J7 732511151, J8 M20-9990445, U5 STM32C071G8Ux, Y1 38.4MHz

Commit message: layout complete
Parts:
- removed C1, C10, C18, C19, C2, C23, C24, C29, C30, C31, C33, C34: 10uF, ar_passives:C_0402, symbol #bt-db:capacitor/CAPC-00667
- removed C39: 100nF, ar_passives:C_0402, symbol #bt-db:capacitor/CAPC-00573
- removed CLF2: 10nF, ar_passives:C_0805, symbol #bt-db:capacitor/CAPC-00850
- removed D6: RG, ar_opto:APHB1608GR, symbol #bt-db:optical/LEDO-00009
- removed H1, H2, H3, H4, H5, H6, H7, H8, H9: GND, MountingHole:MountingHole_2.7mm_M2.5_Pad_Via, symbol Mechanical:MountingHole_Pad
- removed J10: TC2030-NL-FP, ar_connector:TC2030-xxx-NL, symbol #bt-db:connector/CONN-00155
- removed U2: (no value), ar_ic:DFN6-1.55x1.75, symbol #bt-db:ic/ICIR-00298
- added C22: 100nF, ar_passives:C_0402, symbol #bt-db:capacitor/CAPC-00573
- added C25, C8: 10uF, ar_passives:C_0402, symbol #bt-db:capacitor/CAPC-00667
- added C26, C27, C28, C29, C30, C31, C32, C33, C35, C38: 10uF, ar_passives:C_0805, symbol #bt-db:capacitor/CAPC-00926
- added C5: 47nF, ar_passives:C_1206, symbol #bt-db:capacitor/CAPC-00964
- added D3: Green, ar_opto:LED_0603, symbol #bt-db:optical/LEDO-00006
- added D4: Red, ar_opto:LED_0603, symbol #bt-db:optical/LEDO-00004
- added J5: FTSH-105-01-L-DV-K, ar_connector:FTSH-105-01-X-DV-K, symbol #bt-db:connector/CONN-00005
- added TP2: MUX, ar_non-bom:Testpad_1mm, symbol Connector:TestPoint
- added U4: (no value), ar_ic:DFN6-1.55x1.75, symbol #bt-db:ic/ICIR-00298
- TP1: value SDA -> SCK
- TP10: value CE -> SDA
- TP11: value CS -> SDA
- TP3: value SDA -> SDI
- TP4: value SCL -> RC
- TP5: value SCK -> RD
- TP6: value MUX -> CE
- TP7: value SDI -> CS
- TP8: value RC -> SCL
- TP9: value RD -> SDA
- renumbered C27 to C1, C11 to C10, C12 to C11, C13 to C12, C14 to C13, C15 to C14, C21 to C15, C7 to C16, C8 to C17, C16 to C18, C17 to C19, C28 to C2, C36 to C20, C37 to C21, C6 to C23, C5 to C24, C35 to C34, C26 to C36, C38 to C37, C20 to C39, C25 to C40, C32 to C7, CLF3 to CLF1, CLF1 to CLF3, D2 to D1, D3 to D2, D1 to D5, J2 to J1, J3 to J2, J4 to J3, J5 to J4, J1 to J6, J6 to J8, J8 to J9, R9 to R1, R2 to R10, R19 to R11, R20 to R12, R21 to R13, R22 to R14, R3 to R15, R4 to R16, R11 to R17, R12 to R18, R14 to R19, R5 to R2, R13 to R20, R18 to R21, R17 to R22, R10 to R3, R6 to R4, R7 to R5, R8 to R6, R15 to R7, R16 to R8, R1 to R9, RLF1 to RLF3, U4 to U1, U5 to U2, U1 to U3, U3 to U6, Y1 to Y2
Connections:
- net 3V3_BUCK: now also R17.1, C26.1, C28.1, C29.1, C30.1; no longer C4.1, C9.1
- net 3V3_BUF: now also C33.1
- net 3V3_MCU: now also C22.1, C32.1, J5.1; no longer R17.1
- net 3V3_OSC: now also C35.1
- net 3V3_SYN: now also C38.1
- net BUCK_EN: now also U2.14 (PB0); no longer U2.17 (PC6)
- net CON_DN: now also U4.6 (IC+)
- net CON_DP: now also U4.5 (IC-)
- net DBG_RX: now also TP10.1, U2.7 (PA1), J5.8
- net DBG_SWCLK: now also J5.4
- net DBG_SWDIO: now also J5.2
- net DBG_TX: now also TP11.1, U2.6 (PA0), J5.6; no longer TP1.1, U2.26 (PB6)
- net GND: now also C22.2, C25.2, C26.2, C27.2, C28.2, C29.2, C30.2, C31.2, C32.2, C33.2, C35.2, C38.2, C5.2, C8.2, D3.K, D4.K, J5.3, J5.5, J5.7, J5.9, U4.3 (GND)
- net LED_ERR: now also U2.10 (PA4); no longer U2.1 (PC14)
- net LED_STAT: now also U2.9 (PA3); no longer U2.28 (PB8)
- net OLED_SCL: now also TP8.1, U2.13 (PA7); no longer TP3.1, U2.23 (PB3)
- net OLED_SDA: now also TP9.1, U2.12 (PA6); no longer TP4.1, U2.24 (PB4)
- net SYN.CE: now also TP6.1, U2.28 (PB8); no longer TP10.1, U2.12 (PA6)
- net SYN.MUX: now also U2.24 (PB4), TP2.1; no longer TP6.1, U2.7 (PA1)
- net SYN.RC: now also TP4.1, U2.26 (PB6); no longer TP9.1, U2.15 (PB1)
- net SYN.RD: now also TP5.1, U2.27 (PB7); no longer TP8.1, U2.14 (PB0)
- net SYN.SCK: now also TP1.1, U2.23 (PB3); no longer TP5.1, U2.11 (PA5)
- net SYN.SDI: now also TP3.1, U2.25 (PB5); no longer TP7.1, U2.8 (PA2)
- net SYN.~{CS}: now also TP7.1, U2.22 (PA15); no longer TP11.1, U2.16 (PA8)
- net USB_DN: now also U4.1 (CON+)
- net USB_DP: now also U4.2 (CON-)
- net VBUS: now also C27.1, C31.1; no longer C3.1
- net VbiasVARAC: now also C4.1
- net VbiasVCO: now also C9.1
- net VbiasVCO2: now also C25.1
- net VrefVCO: now also C3.1
- net VrefVCO2: now also C8.1
- net ~{DBG_NRST}: now also J5.10
- net at R13.2: now also D3.A
- net at R14.2: now also D4.A
- net at RLF2.2: now also C5.1
- new net MCU_REF_IN: U2.1 (PC14)
- no-connect marks 14 -> 6
